File: pcb/peautkb.sch (KiCad schematic (older format))
At the start: 234 parts, among them J1 Conn_01x04, J2 MJ-4PP-9, J3 Conn_01x04, J4 MJ-4PP-9, SW10 SW_PUSH, SW11 SW_PUSH, SW12 SW_PUSH, SW13 SW_PUSH, SW14 SW_PUSH, SW15 SW_PUSH, SW16 SW_PUSH, SW17 SW_PUSH, SW18 SW_PUSH, SW19 SW_PUSH, SW20 SW_PUSH, SW21 SW_PUSH, SW22 SW_PUSH, SW23 SW_PUSH, SW24 SW_PUSH, SW25 SW_PUSH, SW26 SW_PUSH, SW27 SW_PUSH, SW28 Rotary_Encoder_Switch, SW29 SW_PUSH, SW33 SW_PUSH, SW34 SW_PUSH, SW35 SW_PUSH, SW36 SW_PUSH, SW37 SW_PUSH, SW38 SW_PUSH, SW39 SW_PUSH, SW4 SW_PUSH, SW40 SW_PUSH, SW41 SW_PUSH, SW42 SW_PUSH, SW43 SW_PUSH, SW44 SW_PUSH, SW45 SW_PUSH, SW46 SW_PUSH, SW47 SW_PUSH, SW48 SW_PUSH, SW49 SW_PUSH, SW5 SW_PUSH, SW50 SW_PUSH, SW51 SW_PUSH, SW52 SW_PUSH, SW53 SW_PUSH, SW54 SW_PUSH, SW55 SW_PUSH, SW56 SW_PUSH, SW57 Rotary_Encoder_Switch, SW58 SW_PUSH, SW6 SW_PUSH, SW7 SW_PUSH, SW8 SW_PUSH, SW9 SW_PUSH, U1 black-pill-v3, U2 black-pill-v3

Commit message: updated rotary encoder pins to avoid crystal
Connections:
- net LENCA: now also U1.12 (PB4); no longer U1.23 (PC14)
- net LENCB: now also U1.13 (PB5); no longer U1.22 (PC13)
Changed lines of the file:
@@
 Wire Wire Line
 	3255 9665 3495 9665
-Text GLabel 3610 10355 2    50   Input ~ 0
+Text GLabel 2195 9465 0    50   Input ~ 0
 LENCA
-Text GLabel 3610 10460 2    50   Input ~ 0
+Text GLabel 2195 9575 0    50   Input ~ 0
 LENCB
-Wire Wire Line
-	3255 10040 3435 10040
-Wire Wire Line
-	3435 10040 3435 10355
-Wire Wire Line
-	3435 10355 3610 10355
-Wire Wire Line
-	3255 10115 3420 10115
-Wire Wire Line
-	3420 10115 3420 10460
-Wire Wire Line
-	3420 10460 3610 10460
 $Comp
 L peautkb:black-pill-v3 U1
@@
 NoConn ~ 2355 9365
 NoConn ~ 2355 9440
-Text GLabel 2150 9515 0    50   Input ~ 0
+Text GLabel 2195 9350 0    50   Input ~ 0
 LLED_In
-NoConn ~ 2355 9590
-NoConn ~ 2355 9665
 NoConn ~ 2355 9890
 NoConn ~ 2355 9965
-Wire Wire Line
-	2355 9515 2150 9515
 Wire Wire Line
 	9025 8685 9155 8685
@@
 Wire Wire Line
 	9340 9330 9385 9330
+Wire Wire Line
+	2355 9515 2275 9515
+Wire Wire Line
+	2275 9515 2275 9350
+Wire Wire Line
+	2275 9350 2195 9350
+Wire Wire Line
+	2355 9590 2255 9590
+Wire Wire Line
+	2255 9590 2255 9465
+Wire Wire Line
+	2255 9465 2195 9465
+Wire Wire Line
+	2355 9665 2235 9665
+Wire Wire Line
+	2235 9665 2235 9575
+Wire Wire Line
+	2235 9575 2195 9575
+NoConn ~ 3255 10040
+NoConn ~ 3255 10115
 $EndSCHEMATC

Commit message: before 4->2 layer rework
Connections:
- net RENCA: now also U2.12 (PB4); no longer U2.23 (PC14)
- net RENCB: now also U2.13 (PB5); no longer U2.22 (PC13)
- net VCC: no longer J3.3 (Pin_3)
- net VDD: no longer J1.3 (Pin_3)
- net +3V0: now reaches U1.20 (3V3)
- net +3V0: now also J1.3 (Pin_3)
- net +3V3: now reaches U2.20 (3V3)
- net +3V3: now also J3.3 (Pin_3)
- no-connect marks 40 -> 38
Changed lines of the file:
@@
 	2240 10115 2240 10395
 NoConn ~ 3255 8915
-NoConn ~ 2355 10190
 NoConn ~ 3255 10190
 $Comp
@@
 	1    4670 9475
 	0    -1   -1   0
-$EndComp
-$Comp
-L power:VDD #PWR0128
-U 1 1 6147ED9F
-P 4670 9575
-F 0 "#PWR0128" H 4670 9425 50  0001 C CNN
-F 1 "VDD" V 4685 9703 50  0000 L CNN
-F 2 "" H 4670 9575 50  0001 C CNN
-F 3 "" H 4670 9575 50  0001 C CNN
-	1    4670 9575
-	0    1    1    0
 $EndComp
 Text GLabel 4670 9675 2    50   Input ~ 0
@@
 	8010 10035 8010 10315
 NoConn ~ 9025 8835
-NoConn ~ 8125 10110
 NoConn ~ 9025 10110
 $Comp
@@
 Wire Wire Line
 	9250 9960 9380 9960
-Text GLabel 9380 10275 2    50   Input ~ 0
+Text GLabel 7905 9405 0    50   Input ~ 0
 RENCA
-Text GLabel 9380 10380 2    50   Input ~ 0
+Text GLabel 7910 9515 0    50   Input ~ 0
 RENCB
-Wire Wire Line
-	9025 9960 9205 9960
-Wire Wire Line
-	9205 9960 9205 10275
-Wire Wire Line
-	9205 10275 9380 10275
-Wire Wire Line
-	9025 10035 9190 10035
-Wire Wire Line
-	9190 10035 9190 10380
-Wire Wire Line
-	9190 10380 9380 10380
 $Comp
 L peautkb:black-pill-v3 U2
@@
 NoConn ~ 8125 9285
 NoConn ~ 8125 9360
-Text GLabel 7920 9435 0    50   Input ~ 0
+Text GLabel 7905 9290 0    50   Input ~ 0
 RLED_In
-NoConn ~ 8125 9510
-NoConn ~ 8125 9585
 NoConn ~ 8125 9810
 NoConn ~ 8125 9885
-Wire Wire Line
-	8125 9435 7920 9435
 $Comp
 L power:VCC #PWR0129
@@
 Wire Wire Line
 	9155 8585 9155 8685
-$Comp
-L power:VCC #PWR0130
-U 1 1 621EB59E
-P 10440 9495
-F 0 "#PWR0130" H 10440 9345 50  0001 C CNN
-F 1 "VCC" V 10455 9623 50  0000 L CNN
-F 2 "" H 10440 9495 50  0001 C CNN
-F 3 "" H 10440 9495 50  0001 C CNN
-	1    10440 9495
-	0    1    1    0
-$EndComp
 $Comp
 L power:GND2 #PWR0131
@@
 NoConn ~ 3255 10040
 NoConn ~ 3255 10115
+Wire Wire Line
+	8125 9435 8020 9435
+Wire Wire Line
+	8020 9435 8020 9290
+Wire Wire Line
+	8020 9290 7905 9290
+Wire Wire Line
+	8125 9510 7990 9510
+Wire Wire Line
+	7990 9510 7990 9405
+Wire Wire Line
+	7990 9405 7905 9405
+Wire Wire Line
+	8125 9585 7965 9585
+Wire Wire Line
+	7965 9585 7965 9515
+Wire Wire Line
+	7965 9515 7910 9515
+NoConn ~ 9025 9960
+NoConn ~ 9025 10035
+$Comp
+L power:+3V3 #PWR0122
+U 1 1 607C224F
+P 10440 9495
+F 0 "#PWR0122" H 10440 9345 50  0001 C CNN
+F 1 "+3V3" V 10455 9623 50  0000 L CNN
+F 2 "" H 10440 9495 50  0001 C CNN
+F 3 "" H 10440 9495 50  0001 C CNN
+	1    10440 9495
+	0    1    1    0
+$EndComp
+$Comp
+L power:+3V3 #PWR0128
+U 1 1 607C47BB
+P 8125 10110
+F 0 "#PWR0128" H 8125 9960 50  0001 C CNN
+F 1 "+3V3" V 8140 10238 50  0000 L CNN
+F 2 "" H 8125 10110 50  0001 C CNN
+F 3 "" H 8125 10110 50  0001 C CNN
+	1    8125 10110
+	0    -1   -1   0
+$EndComp
+$Comp
+L power:+3V0 #PWR0120
+U 1 1 607CB373
+P 2355 10190
+F 0 "#PWR0120" H 2355 10040 50  0001 C CNN
+F 1 "+3V0" V 2370 10318 50  0000 L CNN
+F 2 "" H 2355 10190 50  0001 C CNN
+F 3 "" H 2355 10190 50  0001 C CNN
+	1    2355 10190
+	0    -1   -1   0
+$EndComp
+$Comp
+L power:+3V0 #PWR0130
+U 1 1 607CCD77
+P 4670 9575
+F 0 "#PWR0130" H 4670 9425 50  0001 C CNN
+F 1 "+3V0" V 4685 9703 50  0000 L CNN
+F 2 "" H 4670 9575 50  0001 C CNN
+F 3 "" H 4670 9575 50  0001 C CNN
+	1    4670 9575
+	0    1    1    0
+$EndComp
 $EndSCHEMATC
