File: pcb/peautkb.kicad_pcb (KiCad board)
At the start: 4 copper layers, 348 x 113 mm, 258 parts, among them J1 Conn_01x04, J2 MJ-4PP-9, J3 Conn_01x04, J4 MJ-4PP-9, SW10 SW_PUSH, SW11 SW_PUSH, SW12 SW_PUSH, SW13 SW_PUSH, SW14 SW_PUSH, SW15 SW_PUSH, SW16 SW_PUSH, SW17 SW_PUSH, SW18 SW_PUSH, SW19 SW_PUSH, SW20 SW_PUSH, SW21 SW_PUSH, SW22 SW_PUSH, SW23 SW_PUSH, SW24 SW_PUSH, SW25 SW_PUSH, SW26 SW_PUSH, SW27 SW_PUSH, SW28 Rotary_Encoder_Switch, SW29 SW_PUSH, SW33 SW_PUSH, SW34 SW_PUSH, SW35 SW_PUSH, SW36 SW_PUSH, SW37 SW_PUSH, SW38 SW_PUSH, SW39 SW_PUSH, SW4 SW_PUSH, SW40 SW_PUSH, SW41 SW_PUSH, SW42 SW_PUSH, SW43 SW_PUSH, SW44 SW_PUSH, SW45 SW_PUSH, SW46 SW_PUSH, SW47 SW_PUSH, SW48 SW_PUSH, SW49 SW_PUSH, SW5 SW_PUSH, SW50 SW_PUSH, SW51 SW_PUSH, SW52 SW_PUSH, SW53 SW_PUSH, SW54 SW_PUSH, SW55 SW_PUSH, SW56 SW_PUSH, SW57 Rotary_Encoder_Switch, SW58 SW_PUSH, SW6 SW_PUSH, SW7 SW_PUSH, SW8 SW_PUSH, SW9 SW_PUSH, U1 black-pill-v3, U2 black-pill-v3

Commit message: added practice pads
Parts:
- added C9: 100nF, Capacitor_SMD:C_0805_2012Metric_Pad1.18x1.45mm_HandSolder, F.Cu at (47.0, 110.0)
- added C9: 100nF, Capacitor_SMD:C_0805_2012Metric_Pad1.18x1.45mm_HandSolder, F.Cu at (25.0, 110.0)
- added C9: 100nF, Capacitor_SMD:C_0805_2012Metric_Pad1.18x1.45mm_HandSolder, F.Cu at (69.0, 110.0)
- added C9: 100nF, Capacitor_SMD:C_0805_2012Metric_Pad1.18x1.45mm_HandSolder, F.Cu at (58.0, 110.0)
- added C9: 100nF, Capacitor_SMD:C_0805_2012Metric_Pad1.18x1.45mm_HandSolder, F.Cu at (36.0, 110.0)
- added D12: D, kbd:D3_SMD_v2, F.Cu at (322.5, 109.6)
- added D12: D, kbd:D3_SMD_v2, F.Cu at (305.0, 109.6)
- added D12: D, kbd:D3_SMD_v2, F.Cu at (333.0, 109.6)
- added D12: D, kbd:D3_SMD_v2, F.Cu at (326.0, 109.6)
- added D12: D, kbd:D3_SMD_v2, F.Cu at (329.5, 109.6)
- added D12: D, kbd:D3_SMD_v2, F.Cu at (336.5, 109.6)
- added D12: D, kbd:D3_SMD_v2, F.Cu at (319.0, 109.6)
- added D12: D, kbd:D3_SMD_v2, F.Cu at (315.5, 109.6)
- added D12: D, kbd:D3_SMD_v2, F.Cu at (312.0, 109.6)
- added D12: D, kbd:D3_SMD_v2, F.Cu at (308.5, 109.6)
- added D5: SK6812, LED_SMD:LED_SK6812_PLCC4_5.0x5.0mm_P3.2mm, F.Cu at (74.5, 110.5)
- added D5: SK6812, LED_SMD:LED_SK6812_PLCC4_5.0x5.0mm_P3.2mm, F.Cu at (63.5, 110.5)
- added D5: SK6812, LED_SMD:LED_SK6812_PLCC4_5.0x5.0mm_P3.2mm, F.Cu at (52.5, 110.5)
- added D5: SK6812, LED_SMD:LED_SK6812_PLCC4_5.0x5.0mm_P3.2mm, F.Cu at (41.5, 110.5)
- added D5: SK6812, LED_SMD:LED_SK6812_PLCC4_5.0x5.0mm_P3.2mm, F.Cu at (30.5, 110.5)
- added REF**: PinHeader_1x03_P2.54mm_Vertical, Connector_PinHeader_2.54mm:PinHeader_1x03_P2.54mm_Vertical, F.Cu at (20.5, 113.5)
Routing:
- net (no net): track 0.00 -> 215.0 mm, vias 0 -> 10
Other:
- board text added: "5v"
- board text added: "GND"

Commit message: logo and final OLED placement
Parts:
- added G***: LOGO, peautkb:logo, F.Cu at (65.0, 86.0)
- added G***: LOGO, peautkb:logo, F.Cu at (306.1, 85.9)
- moved J1 8.54 mm to (177.2, 65.6)
- moved J3 8.47 mm to (194.2, 58.0)
- moved Ref** 6.40 mm to (64.9, 91.5)
- moved Ref** 4.34 mm to (306.1, 91.5)
Routing:
- net RUSART_RX: track 53.7 -> 68.6 mm
- net LSCA: track 38.4 -> 47.0 mm
- net LSCL: track 42.1 -> 50.1 mm
- net RSCA: track 6.18 -> 13.4 mm
- net RSCL: track 6.18 -> 8.38 mm
- net Net-(LED28-Pad2): track 59.0 -> 59.8 mm
Other:
- board text added: "peautkb v1.0"

Commit message: pcb tweaks
Parts:
- removed the Ref** at (194.0, 48.0)
- removed the Ref** at (177.9, 48.0)
- removed the Ref** at (161.2, 86.2)
- removed the Ref** at (209.7, 86.1)
- added Ref**: Val**, kbd:M2_HOLE_v2, F.Cu at (194.0, 43.8)
- added Ref**: Val**, kbd:M2_HOLE_v2, F.Cu at (177.9, 43.8)
- added Ref**: Val**, kbd:M2_HOLE_v2, F.Cu at (172.2, 87.2)
- added Ref**: Val**, kbd:M2_HOLE_v2, F.Cu at (199.2, 87.2)
Routing:
- net RUSART_RX: track 68.6 -> 54.7 mm
Changed lines of the file:
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@@
     (thickness 1.6)
     (drawings 343)
-    (tracks 2034)
+    (tracks 2033)
     (zones 0)
     (modules 281)
@@
   )
   (module kbd:M2_HOLE_v2 (layer F.Cu)
-    (at 194 48)
+    (at 194 43.75)
     (descr "Mounting Hole 2.2mm, no annular, M2")
     (tags "mounting hole 2.2mm no annular m2")
@@
   )
   (module kbd:M2_HOLE_v2 (layer F.Cu)
-    (at 177.9 48)
+    (at 177.9 43.75)
     (descr "Mounting Hole 2.2mm, no annular, M2")
     (tags "mounting hole 2.2mm no annular m2")
@@
   )
   (module kbd:M2_HOLE_v2 (layer F.Cu)
-    (at 161.2 86.2)
+    (at 172.25 87.25)
     (descr "Mounting Hole 2.2mm, no annular, M2")
     (tags "mounting hole 2.2mm no annular m2")
@@
   )
   (module kbd:M2_HOLE_v2 (layer F.Cu)
-    (at 209.7 86.1)
+    (at 199.25 87.25)
     (descr "Mounting Hole 2.2mm, no annular, M2")
     (tags "mounting hole 2.2mm no annular m2")
@@
   (segment (start 203.332578 89.241637) (end 203.332578 91.883749) (width 0.25) (layer B.Cu) (net 86))
   (segment (start 203.072075 88.981134) (end 203.332578 89.241637) (width 0.25) (layer B.Cu) (net 86))
-  (segment (start 193.25 79.159059) (end 203.072075 88.981134) (width 0.25) (layer B.Cu) (net 86))
   (segment (start 200.19492 48.6438) (end 192 56.83872) (width 0.25) (layer B.Cu) (net 86))
-  (segment (start 192 77.909059) (end 203.072075 88.981134) (width 0.25) (layer B.Cu) (net 86))
   (segment (start 192 56.83872) (end 192 77.909059) (width 0.25) (layer B.Cu) (net 86))
+  (segment (start 192 77.909059) (end 203.072075 88.981134) (width 0.25) (layer B.Cu) (net 86))
   (segment (start 200.19492 76.5838) (end 205.25 81.63888) (width 0.5) (layer B.Cu) (net 87))
   (segment (start 205.25 89.818997) (end 205.198441 89.870556) (width 0.5) (layer B.Cu) (net 87))

Commit message: updated rotary encoder pins to avoid crystal
Parts:
- removed the D12 at (305.0, 109.6)
- removed the D12 at (319.0, 109.6)
- removed the D12 at (315.5, 109.6)
- removed the D12 at (312.0, 109.6)
- removed the D12 at (308.5, 109.6)
- removed the D5 at (52.5, 110.5)
- removed the D5 at (41.5, 110.5)
- removed the D5 at (30.5, 110.5)
- added T1: SK6812, LED_SMD:LED_SK6812_PLCC4_5.0x5.0mm_P3.2mm, F.Cu at (30.5, 110.5)
- added T2: SK6812, LED_SMD:LED_SK6812_PLCC4_5.0x5.0mm_P3.2mm, F.Cu at (41.5, 110.5)
- added T3: SK6812, LED_SMD:LED_SK6812_PLCC4_5.0x5.0mm_P3.2mm, F.Cu at (52.5, 110.5)
- added TD1: D, kbd:D3_SMD_v2, F.Cu at (305.0, 109.6)
- added TD2: D, kbd:D3_SMD_v2, F.Cu at (308.5, 109.6)
- added TD3: D, kbd:D3_SMD_v2, F.Cu at (312.0, 109.6)
- added TD4: D, kbd:D3_SMD_v2, F.Cu at (315.5, 109.6)
- added TD5: D, kbd:D3_SMD_v2, F.Cu at (319.0, 109.6)
- renumbered C9 to CT1, C9 to CT2, C9 to CT3, C9 to CT4, C9 to CT5, D5 to T4, D5 to T5, D12 to TD10, D12 to TD6, D12 to TD7, D12 to TD8, D12 to TD9
Connections:
- U1 pad 12: Net-(U1-Pad12) -> LENCA
- U1 pad 13: Net-(U1-Pad13) -> LENCB
- U1 pad 22: LENCB -> Net-(U1-Pad22)
- U1 pad 23: LENCA -> Net-(U1-Pad23)
- U2 pad 12: Net-(U2-Pad12) -> RENCA
- U2 pad 13: Net-(U2-Pad13) -> RENCB
- U2 pad 22: RENCB -> Net-(U2-Pad22)
- U2 pad 23: RENCA -> Net-(U2-Pad23)
Routing:
- net RENCB: track 25.7 -> 53.5 mm, vias 0 -> 1
- net RENCA: track 23.3 -> 48.1 mm, vias 1 -> 0
- net LENCA: track 46.5 -> 26.3 mm
- net LENCB: track 47.5 -> 28.9 mm
- net Net-(LED28-Pad2): track 59.8 -> 61.1 mm
- net (no net): track 215.0 -> 213.7 mm, vias 10 -> 9

Commit message: before 4->2 layer rework
Parts:
- added Ref**: Val**, kbd:M2_HOLE_v2, F.Cu at (277.5, 22.5)
- added Ref**: Val**, kbd:M2_HOLE_v2, F.Cu at (94.0, 22.5)
Connections:
- J1 pad 3: VDD -> +3V0
- J3 pad 3: VCC -> +3V3
- U1 pad 20: Net-(U1-Pad20) -> +3V0
- U2 pad 20: Net-(U2-Pad20) -> +3V3
Routing:
- net +3V0: track 0.00 -> 43.8 mm
- net +3V3: track 0.00 -> 21.0 mm

Commit message: re-worked with copper pours for gnd and 5v routed, re-routed the LHS completely
Parts:
- removed CT1, CT2, CT3, CT4, CT5: 100nF, Capacitor_SMD:C_0805_2012Metric_Pad1.18x1.45mm_HandSolder
- removed the REF** at (20.5, 113.5)
- removed T1, T2, T3, T4, T5: SK6812, LED_SMD:LED_SK6812_PLCC4_5.0x5.0mm_P3.2mm
- removed TD1, TD10, TD2, TD3, TD4, TD5, TD6, TD7, TD8, TD9: D, kbd:D3_SMD_v2
- moved LED22 0.41 mm to (141.0, 102.8)
Routing:
- net VCC: track 101.2 -> 872.2 mm, vias 31 -> 38
- net VDD: track 99.0 -> 840.1 mm, vias 31 -> 40
- net (no net): track 213.7 -> 0.00 mm, vias 9 -> 0
- net LCol6: track 182.3 -> 134.0 mm, vias 7 -> 8
- net LCol5: track 196.7 -> 152.5 mm, vias 7 -> 8
- net LCol2: track 218.8 -> 181.7 mm, vias 6 -> 4
- net LCol4: track 218.1 -> 181.8 mm
- net LCol7: track 154.5 -> 126.4 mm, vias 7 -> 5
- net LSCL: track 50.1 -> 22.5 mm
- net LCol3: track 228.8 -> 201.2 mm
- net LRow0: track 185.0 -> 158.9 mm, vias 0 -> 2
- net LCol1: track 231.6 -> 205.7 mm, vias 0 -> 4
- net LSCA: track 47.0 -> 22.5 mm
- net LRow1: track 194.5 -> 171.3 mm, vias 2 -> 4
- net GND1: track 107.3 -> 88.6 mm
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- added copper zone on B.Cu, net GND1
- added copper zone on F.Cu, net GND1
- added copper zone on B.Cu, net GND2
- added copper zone on F.Cu, net GND2
- removed copper zone on In1.Cu, net GND1
- removed copper zone on In1.Cu, net GND2
- removed copper zone on In2.Cu, net VCC
- removed copper zone on In2.Cu, net VDD
Other:
- copper layers 4 -> 2
- board text removed: "5v"
- board text removed: "GND"

Commit message: submitted pcbs - i hope
Parts:
- removed G*** (x2): LOGO, peautkb:logo
